Commit message: 2/12/22

File: extrernal_urdfs/aruco.xacro (robot description, xacro)
@@ -1,7 +1,7 @@
 <?xml version="1.0"?>
 <robot xmlns:xacro="http://ros.org/wiki/xacro">
-  <joint name="aruco_joint" type="fixed">
+  <joint name="camera_joint" type="fixed">
       <axis xyz="0 1 0" />
-      <origin rpy="0 ${pi/2} 0" xyz="0 0.0 0.0025" />
+      <origin rpy="0 ${pi/2} 0" xyz="0 0.54 0.8" />
       <!--parent link fixed-->
       <parent link="$(arg robot_name)/base_link"/>
@@ -38,4 +38,67 @@
   <gazebo reference="camera_link">
      <material>Gazebo/Red</material>
+     <sensor type="camera" name="camera">
+        <pose>0 0 0 0 0 0</pose>
+        <always_on>true</always_on>
+        <visualize>true</visualize>
+        <update_rate>10</update_rate>
+        <camera>
+          <horizontal_fov>1.5</horizontal_fov>
+          <image>
+            <format>R8G8B8</format>
+            <width>640</width>
+            <height>480</height>
+          </image>
+          <clip>
+            <near>0.05</near>
+            <far>8.0</far>
+          </clip>
+        </camera>
+        <plugin filename="libgazebo_ros_camera.so" name="camera_controller">
+          <cameraName>camera_link_optical</cameraName>
+          <frameName>camera_link_optical</frameName>
+          <!-- <topic_name>/ws200/image_raw</topic_name> -->
+          <!-- <frame_name>camera_link_optical</frame_name> -->
+        </plugin>
+    </sensor>
   </gazebo>
+<!-- aruco marker link -->
+<joint name="camera_joint" type="fixed">
+    <axis xyz="0 1 0" />
+    <origin rpy="0 ${pi/2} 0" xyz="0 0.54 0.8" />
+    <!--parent link fixed-->
+    <parent link="$(arg robot_name)/base_link"/>
+    <child link="camera_link"/>
+</joint>
+<link name="camera_link">
+  <visual>
+    <origin xyz="0 0 0" rpy="0 0 0"/>
+    <geometry>
+      <box size="0.01 0.03 0.03"/>
+    </geometry>
+    <!-- <material name="red"/> -->
+  </visual>
+  <collision>
+    <origin xyz="0 0 0" rpy="0 0 0"/>
+    <geometry>
+      <box size="0.01 0.01 0.01"/>
+    </geometry>
+  </collision>
+  <inertial>
+    <mass value="1e-5" />
+    <origin xyz="0 0 0" rpy="0 0 0"/>
+    <inertia ixx="1e-6" ixy="0" ixz="0" iyy="1e-6" iyz="0" izz="1e-6" />
+  </inertial>
+</link>
+<joint name="camera_optical_joint" type="fixed">
+    <axis xyz="0 1 0" />
+    <!--This is to go from ros image coordinates to common visual coordinates-->
+    <origin rpy="${-pi/2} 0 ${-pi/2}" xyz="0 0 0" />
+    <parent link="camera_link"/>
+    <child link="camera_link_optical"/>
+</joint>
+<link name="camera_link_optical"></link>
+<gazebo reference="camera_link">
+   <material>Gazebo/Red</material>
+</gazebo>
 </robot>
